File: High Power Rocket Flight Computer/KiCad Project/KiCad Project.kicad_sch (KiCad schematic)
At the start: 12 parts, among them U1 STM32F103C8T6

Commit message: 2025/11/18
Parts:
- added C12: C, symbol Device:C
- added Y1: ECS-2520MV-160-CN-TR, Oscillator:Oscillator_SMD_ECS_2520MV-xxx-xx-4Pin_2.5x2.0mm, symbol Oscillator:ECS-2520MV-xxx-xx
Connections:
- net +3.3V: now also C12.1, Y1.4 (VDD); no longer C9.1, R1.1
- net GND: now also C12.2, Y1.2 (GND)
- net STM_OSC IN: now reaches U1.5 (PD0)
- net STM_OSC OUT: now reaches U1.6 (PD1)
- net BOOT0 renamed STM_BOOT0
- net ~{RST} renamed STM_~{RST}
- new net: C9.1, R1.1
- new net STM_OSC_IN: Y1.1 (Tri-State)
- new net STM_OSC_OUT: Y1.3 (OUT)
Other:
- moved on the sheet: C9, R1

Commit message: 2025/11/19
Parts:
- added P1: USB_C_Plug_USB2.0, symbol Connector:USB_C_Plug_USB2.0
- added R2: 1k5, symbol Device:R
- C12: value C -> 100n
Connections:
- net +3.3V: now also R2.1
- net GND: now also P1.A1 (GND), P1.A12 (GND), P1.B1 (GND), P1.B12 (GND)
- net STM_USB_D-: now reaches U1.32 (PA11)
- net STM_USB_D-: now also P1.A7 (D-)
- net STM_USB_D+: now reaches U1.33 (PA12)
- net STM_USB_D+: now also P1.A6 (D+), R2.2
- new net STM_USB_CC: P1.A5 (CC)
- new net USB_VCONN: P1.B5 (VCONN)
- new net VBUS: P1.A4 (VBUS), P1.A9 (VBUS), P1.B4 (VBUS), P1.B9 (VBUS)
- no-connect marks 0 -> 1
Other:
- moved on the sheet: C12, Y1
