File: KiCad Project/STMRocket_Sheet4_Datalogging.kicad_sch (KiCad schematic)
At the start: 12 parts, among them J6 Micro_SD_Card, U4 AT25SF041B-SSHD-T, U5 PESD3V3S4UD,115

Commit message: Updated layout, documentation and schematic. Component placement finished.
Parts:
- C12, C20, C21, C22: footprint Capacitor_SMD:C_0603_1608Metric -> Capacitor_SMD:C_0402_1005Metric
- C7: footprint Capacitor_SMD:C_0805_2012Metric -> Capacitor_SMD:C_0603_1608Metric
- renumbered R4 to R3, R5 to R4, R6 to R5, R3 to R6
Connections:
- net STM_MISO: now also U5.4; no longer U5.6
- net STM_MOSI: now also U5.6; no longer U5.4
Changed lines of the file:
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@@
+	)
+	(junction
+		(at 71.12 60.96)
+		(diameter 0)
+		(color 0 0 0 0)
 	)
 	(junction
@@
 	)
 	(junction
-		(at 81.28 60.96)
-		(diameter 0)
-		(color 0 0 0 0)
-	)
-	(junction
 		(at 243.84 59.69)
 		(diameter 0)
@@
 	)
 	(junction
+		(at 81.28 71.12)
+		(diameter 0)
+		(color 0 0 0 0)
+	)
+	(junction
 		(at 74.93 66.04)
 		(diameter 0)
@@
 	(wire
 		(pts
+			(xy 71.12 60.96) (xy 68.58 60.96)
+		)
+		(stroke
+			(width 0)
+			(type default)
+		)
+	)
+	(wire
+		(pts
 			(xy 238.76 39.37) (xy 238.76 41.91)
 		)
@@
 	(wire
 		(pts
-			(xy 81.28 60.96) (xy 68.58 60.96)
-		)
-		(stroke
-			(width 0)
-			(type default)
-		)
-	)
-	(wire
-		(pts
 			(xy 30.48 49.53) (xy 43.18 49.53)
 		)
@@
 	(wire
 		(pts
-			(xy 90.17 60.96) (xy 81.28 60.96)
+			(xy 71.12 60.96) (xy 90.17 60.96)
 		)
 		(stroke
@@
 	(wire
 		(pts
+			(xy 71.12 74.93) (xy 71.12 60.96)
+		)
+		(stroke
+			(width 0)
+			(type default)
+		)
+	)
+	(wire
+		(pts
 			(xy 54.61 34.29) (xy 54.61 36.83)
 		)
@@
 	(wire
 		(pts
-			(xy 58.42 74.93) (xy 68.58 74.93)
+			(xy 58.42 74.93) (xy 71.12 74.93)
 		)
 		(stroke
@@
 	(wire
 		(pts
+			(xy 81.28 71.12) (xy 81.28 85.09)
+		)
+		(stroke
+			(width 0)
+			(type default)
+		)
+	)
+	(wire
+		(pts
 			(xy 193.04 64.77) (xy 198.12 64.77)
 		)
@@
 	(wire
 		(pts
-			(xy 68.58 74.93) (xy 68.58 71.12)
-		)
-		(stroke
-			(width 0)
-			(type default)
-		)
-	)
-	(wire
-		(pts
 			(xy 58.42 80.01) (xy 74.93 80.01)
 		)
@@
 	(wire
 		(pts
+			(xy 81.28 71.12) (xy 90.17 71.12)
+		)
+		(stroke
+			(width 0)
+			(type default)
+		)
+	)
+	(wire
+		(pts
 			(xy 243.84 72.39) (xy 255.27 72.39)
 		)
@@
 	(wire
 		(pts
-			(xy 68.58 71.12) (xy 90.17 71.12)
+			(xy 68.58 71.12) (xy 81.28 71.12)
 		)
 		(stroke
@@
 		(pts
 			(xy 204.47 41.91) (xy 204.47 44.45)
-		)
-		(stroke
-			(width 0)
-			(type default)
-		)
-	)
-	(wire
-		(pts
-			(xy 81.28 85.09) (xy 81.28 60.96)
 		)
 		(stroke
@@
 			)
 		)
-		(property "Footprint" "Capacitor_SMD:C_0603_1608Metric"
+		(property "Footprint" "Capacitor_SMD:C_0402_1005Metric"
 			(at 244.8052 69.85 0)
 			(effects
@@
 		(on_board yes)
 		(dnp no)
-		(property "Reference" "R4"
+		(property "Reference" "R3"
 			(at 193.548 46.99 0)
 			(effects
@@
 			(project "KiCad Project"
 				(path "/fd47649a-639e-448c-bb16-b2061ebe97a0/77d54ba2-ca2c-4a76-8a14-c2168bfad133"
-					(reference "R4")
+					(reference "R3")
 					(unit 1)
 				)
@@
 		(on_board yes)
 		(dnp no)
-		(property "Reference" "R6"
+		(property "Reference" "R5"
 			(at 206.502 46.99 0)
 			(effects
@@
 			(project "KiCad Project"
 				(path "/fd47649a-639e-448c-bb16-b2061ebe97a0/77d54ba2-ca2c-4a76-8a14-c2168bfad133"
-					(reference "R6")
+					(reference "R5")
 					(unit 1)
 				)
@@
 			)
 		)
-		(property "Footprint" "Capacitor_SMD:C_0603_1608Metric"
+		(property "Footprint" "Capacitor_SMD:C_0402_1005Metric"
 			(at 256.2352 69.85 0)
 			(effects
@@
 			)
 		)
-		(property "Footprint" "Capacitor_SMD:C_0603_1608Metric"
+		(property "Footprint" "Capacitor_SMD:C_0402_1005Metric"
 			(at 136.8552 88.9 0)
 			(effects
@@
 		(dnp no)
 		(fields_autoplaced yes)
-		(property "Reference" "R3"
+		(property "Reference" "R6"
 			(at 83.82 45.7199 0)
 			(effects
@@
 			(project "KiCad Project"
 				(path "/fd47649a-639e-448c-bb16-b2061ebe97a0/77d54ba2-ca2c-4a76-8a14-c2168bfad133"
-					(reference "R3")
+					(reference "R6")
 					(unit 1)
 				)
@@
 			)
 		)
-		(property "Footprint" "Capacitor_SMD:C_0805_2012Metric"
+		(property "Footprint" "Capacitor_SMD:C_0603_1608Metric"
 			(at 44.1452 46.99 0)
 			(effects
@@
 		(on_board yes)
 		(dnp no)
-		(property "Reference" "R5"
+		(property "Reference" "R4"
 			(at 200.152 53.34 0)
 			(effects
@@
 			(project "KiCad Project"
 				(path "/fd47649a-639e-448c-bb16-b2061ebe97a0/77d54ba2-ca2c-4a76-8a14-c2168bfad133"
-					(reference "R5")
+					(reference "R4")
 					(unit 1)
 				)
@@
 			)
 		)
-		(property "Footprint" "Capacitor_SMD:C_0603_1608Metric"
+		(property "Footprint" "Capacitor_SMD:C_0402_1005Metric"
 			(at 31.4452 46.99 0)
 			(effects
