File: KiCad Project/STMRocket_Sheet1_MCU.kicad_sch (KiCad schematic)
At the start: 17 parts, among them U1 STM32F103C8T6, Y1 ECS-2520MV-160-CN-TR

Commit message: Updated layout, documentation and schematic. Component placement finished.
Parts:
- added H1, H2, H3, H4, H5: MountingHole, MountingHole:MountingHole_2.2mm_M2, symbol Mechanical:MountingHole
- C10, C11, C13, C14, C15, C16, C17, C18, C27, C28: footprint Capacitor_SMD:C_0603_1608Metric -> Capacitor_SMD:C_0402_1005Metric
- C8: footprint Capacitor_SMD:C_0805_2012Metric -> Capacitor_SMD:C_0603_1608Metric
- renumbered R9 to R7, R10 to R8
Other:
- note added: "PE-0603PFB121ST"

Commit message: PCB update
Connections:
- net IMU_FSYNC: now also U1.40 (PB4); no longer U1.41 (PB5)
- net IMU_INT1: now also U1.41 (PB5); no longer U1.39 (PB3)
- net IMU_INT2: now also U1.39 (PB3); no longer U1.40 (PB4)

Commit message: finished pcb
Connections:
- net IMU_FSYNC: now also U1.39 (PB3); no longer U1.40 (PB4)
- net IMU_INT1: now also U1.40 (PB4); no longer U1.41 (PB5)
- net IMU_INT2: now also U1.41 (PB5); no longer U1.39 (PB3)
- net ~{CS}_FLASH: now also U1.11 (PA1); no longer U1.13 (PA3)
- net ~{CS}_SD: now also U1.18 (PB0); no longer U1.10 (PA0)
- net ~{WP}_FLASH: now also U1.10 (PA0); no longer U1.11 (PA1)
