File: KiCad Project/STMRocket_Sheet2_Power&Connectors.kicad_sch (KiCad schematic)
At the start: 30 parts, among them J1 XT30PW-M, J2 USB_C_Receptacle_USB2.0_16P, J3 PYRO, J4 PYRO ARM, J5 SWD, Q1 GSFC02A05, Q2 FDMC7692, U6 AP63203WU, U7 ESD122DMXR, U8 ESD122DMXR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

Commit message: Datasheet renaming and schematic formatting, text, tables, etc.
Parts:
- renumbered D4 to D3, D6 to D4, D3 to D5, D7 to D6, D5 to D7
Other:
- note added: "R7,8 ~ 1%"
- title: STMRocket - Power -> STMRocket - Power & Connectors
Changed lines of the file:
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@@
 	(paper "A4")
 	(title_block
-		(title "STMRocket - Power")
+		(title "STMRocket - Power & Connectors")
 		(date "2025-12-09")
 		(rev "1")
@@
 		)
 	)
+	(text "R7,8 ~ 1%\n"
+		(exclude_from_sim no)
+		(at 56.388 116.078 0)
+		(effects
+			(font
+				(size 1.27 1.27)
+			)
+		)
+	)
 	(text "USB D+ 1.5k pull-up resistor required in ST AN4879"
 		(exclude_from_sim no)
@@
 		)
 		(instances
-			(project ""
+			(project "KiCad Project"
 				(path "/fd47649a-639e-448c-bb16-b2061ebe97a0/9995a840-2775-49be-9d1b-261554bf1482"
 					(reference "#PWR049")
@@
 		)
 		(instances
-			(project ""
+			(project "KiCad Project"
 				(path "/fd47649a-639e-448c-bb16-b2061ebe97a0/9995a840-2775-49be-9d1b-261554bf1482"
 					(reference "#PWR025")
@@
 		)
 		(instances
-			(project ""
+			(project "KiCad Project"
 				(path "/fd47649a-639e-448c-bb16-b2061ebe97a0/9995a840-2775-49be-9d1b-261554bf1482"
 					(reference "#PWR031")
@@
 		)
 		(instances
-			(project ""
+			(project "KiCad Project"
 				(path "/fd47649a-639e-448c-bb16-b2061ebe97a0/9995a840-2775-49be-9d1b-261554bf1482"
 					(reference "#PWR016")
@@
 		)
 		(instances
-			(project ""
+			(project "KiCad Project"
 				(path "/fd47649a-639e-448c-bb16-b2061ebe97a0/9995a840-2775-49be-9d1b-261554bf1482"
 					(reference "J3")
@@
 		)
 		(instances
-			(project ""
+			(project "KiCad Project"
 				(path "/fd47649a-639e-448c-bb16-b2061ebe97a0/9995a840-2775-49be-9d1b-261554bf1482"
 					(reference "C1")
@@
 		)
 		(instances
-			(project ""
+			(project "KiCad Project"
 				(path "/fd47649a-639e-448c-bb16-b2061ebe97a0/9995a840-2775-49be-9d1b-261554bf1482"
 					(reference "#PWR032")
@@
 		(on_board yes)
 		(dnp no)
-		(property "Reference" "D7"
+		(property "Reference" "D6"
 			(at 255.27 33.02 0)
 			(effects
@@
 			(project "KiCad Project"
 				(path "/fd47649a-639e-448c-bb16-b2061ebe97a0/9995a840-2775-49be-9d1b-261554bf1482"
-					(reference "D7")
+					(reference "D6")
 					(unit 1)
 				)
@@
 		)
 		(instances
-			(project ""
+			(project "KiCad Project"
 				(path "/fd47649a-639e-448c-bb16-b2061ebe97a0/9995a840-2775-49be-9d1b-261554bf1482"
 					(reference "#PWR028")
@@
 		)
 		(instances
-			(project ""
+			(project "KiCad Project"
 				(path "/fd47649a-639e-448c-bb16-b2061ebe97a0/9995a840-2775-49be-9d1b-261554bf1482"
 					(reference "#PWR018")
@@
 		)
 		(instances
-			(project ""
+			(project "KiCad Project"
 				(path "/fd47649a-639e-448c-bb16-b2061ebe97a0/9995a840-2775-49be-9d1b-261554bf1482"
 					(reference "#PWR029")
@@
 		(on_board yes)
 		(dnp no)
-		(property "Reference" "D5"
+		(property "Reference" "D7"
 			(at 237.49 32.512 0)
 			(effects
@@
 			(project "KiCad Project"
 				(path "/fd47649a-639e-448c-bb16-b2061ebe97a0/9995a840-2775-49be-9d1b-261554bf1482"
-					(reference "D5")
+					(reference "D7")
 					(unit 1)
 				)
@@
 		)
 		(instances
-			(project ""
+			(project "KiCad Project"
 				(path "/fd47649a-639e-448c-bb16-b2061ebe97a0/9995a840-2775-49be-9d1b-261554bf1482"
 					(reference "#FLG04")
@@
 		)
 		(instances
-			(project ""
+			(project "KiCad Project"
 				(path "/fd47649a-639e-448c-bb16-b2061ebe97a0/9995a840-2775-49be-9d1b-261554bf1482"
 					(reference "R1")
@@
 		)
 		(instances
-			(project ""
+			(project "KiCad Project"
 				(path "/fd47649a-639e-448c-bb16-b2061ebe97a0/9995a840-2775-49be-9d1b-261554bf1482"
 					(reference "R1")
@@
 		)
 		(instances
-			(project ""
+			(project "KiCad Project"
 				(path "/fd47649a-639e-448c-bb16-b2061ebe97a0/9995a840-2775-49be-9d1b-261554bf1482"
 					(reference "J4")
@@
 		)
 		(instances
-			(project ""
+			(project "KiCad Project"
 				(path "/fd47649a-639e-448c-bb16-b2061ebe97a0/9995a840-2775-49be-9d1b-261554bf1482"
 					(reference "Q2")
@@
 		)
 		(instances
-			(project ""
+			(project "KiCad Project"
 				(path "/fd47649a-639e-448c-bb16-b2061ebe97a0/9995a840-2775-49be-9d1b-261554bf1482"
 					(reference "#PWR020")
@@
 		(on_board yes)
 		(dnp no)
-		(property "Reference" "D6"
+		(property "Reference" "D4"
 			(at 243.84 106.426 0)
 			(effects
@@
 			(project "KiCad Project"
 				(path "/fd47649a-639e-448c-bb16-b2061ebe97a0/9995a840-2775-49be-9d1b-261554bf1482"
-					(reference "D6")
+					(reference "D4")
 					(unit 1)
 				)
@@
 		)
 		(instances
-			(project ""
+			(project "KiCad Project"
 				(path "/fd47649a-639e-448c-bb16-b2061ebe97a0/9995a840-2775-49be-9d1b-261554bf1482"
 					(reference "#PWR034")
@@
 		(on_board yes)
 		(dnp no)
-		(property "Reference" "D4"
+		(property "Reference" "D3"
 			(at 224.79 106.426 0)
 			(effects
@@
 			(project "KiCad Project"
 				(path "/fd47649a-639e-448c-bb16-b2061ebe97a0/9995a840-2775-49be-9d1b-261554bf1482"
-					(reference "D4")
+					(reference "D3")
 					(unit 1)
 				)
@@
 		(on_board yes)
 		(dnp no)
-		(property "Reference" "D3"
+		(property "Reference" "D5"
 			(at 181.61 101.6 0)
 			(effects
@@
 			(project "KiCad Project"
 				(path "/fd47649a-639e-448c-bb16-b2061ebe97a0/9995a840-2775-49be-9d1b-261554bf1482"
-					(reference "D3")
+					(reference "D5")
 					(unit 1)
 				)

Commit message: Updated layout, documentation and schematic. Component placement finished.
Parts:
- removed J2: USB_C_Receptacle_USB2.0_16P, Connector_USB:USB_C_Receptacle_GCT_USB4085, symbol Connector:USB_C_Receptacle_USB2.0_16P
- removed R7, R8: 5k1, Resistor_SMD:R_0402_1005Metric, symbol Device:R
- added J2: USB_B_Micro, Connector_USB:USB_Micro-B_Amphenol_10103594-0001LF_Horizontal, symbol Connector:USB_B_Micro
- added R10: 2R, Package_TO_SOT_THT:TO-220-2_Horizontal_TabDown, symbol Device:R
- C19: footprint Capacitor_SMD:C_0603_1608Metric -> Capacitor_SMD:C_0402_1005Metric
- C5, C6: footprint Capacitor_SMD:C_0805_2012Metric -> Capacitor_SMD:C_0603_1608Metric
- R1: value 1k5 -> 100k
- renumbered R1 to R9
Connections:
- net +7.5V: no longer C1.1, D2.1 (K), J1.P, Q1.2 (D)
- net +BATT: now also Q1.2 (D); no longer Q1.3 (S)
- net GND: now also D4.2 (A), J2.5 (GND)
- net STM_SWCLK: now also J5.2 (Pin_2); no longer J5.3 (Pin_3)
- net STM_SWDIO: now also J5.3 (Pin_3); no longer J5.2 (Pin_2)
- net STM_USB_D+: now also U8.3 (IO2), J2.3 (D+); no longer U8.2 (IO1)
- net STM_USB_D-: now also U8.2 (IO1), J2.2 (D-); no longer U8.3 (IO2)
- net VBUS: now also J2.1 (VBUS)
- net at D3.1 (K), J3.2 (Pin_2): now also R10.2; no longer D4.2 (A), J4.1 (Pin_1)
- new net: C1.1, D2.1 (K), J1.P, Q1.3 (S)
- new net: J4.1 (Pin_1), R10.1
- no-connect marks 3 -> 2
Other:
- note added: "BRL3225T2R2M"
- note added: "Connector - USB 2.0 Type B"
- note added: "MP930-2.00-1%"
- note removed: "Connector - USB 2.0 Type C"
- note removed: "R7,8 ~ 1%"
- moved on the sheet: Q1, R9, U8

Commit message: PCB update
Parts:
- removed J1: XT30PW-M, Connector_AMASS:AMASS_XT30PW-F_1x02_P2.50mm_Horizontal, symbol XT30PW-M:XT30PW-M
- added J1: BATT XT30, Connector_AMASS:AMASS_XT30PW-M_1x02_P2.50mm_Horizontal, symbol Connector:Conn_01x02_Pin
Connections:
- net +7.5V: now also C1.1, D2.1 (K), Q1.3 (S), J1.2 (Pin_2)
- net GND: now also J1.1 (Pin_1)

Commit message: finished pcb
Parts:
- J1, J3, J4, J5, R10: now not fitted
Changed lines of the file:
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@@
 		(in_bom yes)
 		(on_board yes)
-		(dnp no)
+		(dnp yes)
 		(fields_autoplaced yes)
 		(property "Reference" "J3"
@@
 		(in_bom yes)
 		(on_board yes)
-		(dnp no)
+		(dnp yes)
 		(property "Reference" "J1"
 			(at 38.735 34.29 0)
@@
 		(in_bom yes)
 		(on_board yes)
-		(dnp no)
+		(dnp yes)
 		(fields_autoplaced yes)
 		(property "Reference" "J5"
@@
 		(in_bom yes)
 		(on_board yes)
-		(dnp no)
+		(dnp yes)
 		(property "Reference" "R10"
 			(at 234.95 96.52 90)
@@
 		(in_bom yes)
 		(on_board yes)
-		(dnp no)
+		(dnp yes)
 		(property "Reference" "J4"
 			(at 240.792 107.442 90)
