File: STMRocket - EDA/STMRocket - KiCad Project/STMRocket.kicad_sch (KiCad schematic)
At the start: 0 parts

Commit message: pcb update and bom
Parts:
- added H1, H2, H3, H4, H5: MountingHole, MountingHole:MountingHole_2.2mm_M2, symbol Mechanical:MountingHole
Other:
- note added: "PCB Mounting Holes"
- note added: "Project Description This is a personal project for an STM32 flight computer that will be flown on a high power rocket to acheive the Level 1 high power rocketry certification. Further details are available in the repository: https://github.com/esicoe/STMRocket Capabilities The computer is able to store flight data from it's two sensors: - ICM42670: 6-axis IMU with a gryroscope and accelerometer. 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"
- note removed: "- 4 Mb of NOR flash over 3-wire SPI at 1 MHz. - MicroSD connector for extracting memory from flash IC."
- note removed: "- IMU IC (Intertial measurement unit) containing a programmable gyroscope, accelerometer, and a digital low pass filter. Operates over I2C at 100 KHz with address 0x68. - Environmental sensor IC containing a programmable pressure, humidity, and temperature measurements with a filter. Operates over I2C at 100 KHz with address 0x76."
- note removed: "Project Description This is a personal project for an STM32 flight computer that will be flown on a model rocket to acheive the Level 1 high power rocketry certification. It is open source with details available on the Github repository. https://github.com/esicoe/STMRocket Capabilities The flight computer is able to log flight condition data, including pressure, altitude, acceleration, gyroscope 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"
- note removed: "Revision History"
