File: STMRocket - EDA/STMRocket - KiCad Project/STMRocket_Sheet1_MCU.kicad_sch (KiCad schematic)
At the start: 22 parts, among them U1 STM32F103C8T6, Y1 ECS-2520MV-160-CN-TR

Commit message: pcb update and bom
Parts:
- removed H1, H2, H3, H4, H5: MountingHole, MountingHole:MountingHole_2.2mm_M2, symbol Mechanical:MountingHole
Connections:
- net GND: no longer C13.1
- net IMU_FSYNC: now also U1.40 (PB4); no longer U1.39 (PB3)
- net IMU_INT1: now also U1.41 (PB5); no longer U1.40 (PB4)
- net IMU_INT2: now also U1.39 (PB3); no longer U1.41 (PB5)
- net at R2.2, U1.44 (BOOT0): now also C13.1
Other:
- note removed: "PCB Mounting Holes"
- moved on the sheet: C13
