File: STMRocket - EDA/STMRocket - KiCad Project/STMRocket_Sheet4_Datalogging.kicad_sch (KiCad schematic)
At the start: 12 parts, among them J6 Micro_SD_Card, U4 AT25SF041B-SSHD-T, U5 PESD3V3S4UD,115

Commit message: pcb update and bom
Connections:
- net +3.3V: now also U5.5; no longer U5.3
- net STM_MISO: now also U5.3; no longer U5.4
- net STM_SCK: now also U5.4; no longer U5.5
Changed lines of the file:
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@@
+	)
+	(junction
+		(at 81.28 66.04)
+		(diameter 0)
+		(color 0 0 0 0)
 	)
 	(junction
@@
 	)
 	(junction
+		(at 74.93 63.5)
+		(diameter 0)
+		(color 0 0 0 0)
+	)
+	(junction
 		(at 204.47 41.91)
 		(diameter 0)
@@
 	)
 	(junction
-		(at 54.61 63.5)
-		(diameter 0)
-		(color 0 0 0 0)
-	)
-	(junction
 		(at 243.84 59.69)
 		(diameter 0)
@@
 	)
 	(junction
-		(at 81.28 71.12)
-		(diameter 0)
-		(color 0 0 0 0)
-	)
-	(junction
-		(at 74.93 66.04)
-		(diameter 0)
-		(color 0 0 0 0)
-	)
-	(junction
 		(at 204.47 69.85)
+		(diameter 0)
+		(color 0 0 0 0)
+	)
+	(junction
+		(at 78.74 71.12)
 		(diameter 0)
 		(color 0 0 0 0)
@@
 	(wire
 		(pts
-			(xy 54.61 63.5) (xy 90.17 63.5)
+			(xy 81.28 66.04) (xy 90.17 66.04)
+		)
+		(stroke
+			(width 0)
+			(type default)
+		)
+	)
+	(wire
+		(pts
+			(xy 54.61 63.5) (xy 74.93 63.5)
 		)
 		(stroke
@@
 	(wire
 		(pts
-			(xy 74.93 66.04) (xy 68.58 66.04)
-		)
-		(stroke
-			(width 0)
-			(type default)
-		)
-	)
-	(wire
-		(pts
 			(xy 30.48 49.53) (xy 43.18 49.53)
 		)
@@
 	(wire
 		(pts
+			(xy 78.74 71.12) (xy 90.17 71.12)
+		)
+		(stroke
+			(width 0)
+			(type default)
+		)
+	)
+	(wire
+		(pts
+			(xy 78.74 92.71) (xy 78.74 71.12)
+		)
+		(stroke
+			(width 0)
+			(type default)
+		)
+	)
+	(wire
+		(pts
 			(xy 38.1 53.34) (xy 38.1 74.93)
 		)
@@
 	(wire
 		(pts
-			(xy 33.02 63.5) (xy 54.61 63.5)
-		)
-		(stroke
-			(width 0)
-			(type default)
-		)
-	)
-	(wire
-		(pts
 			(xy 71.12 60.96) (xy 90.17 60.96)
 		)
@@
 	(wire
 		(pts
-			(xy 74.93 80.01) (xy 74.93 66.04)
-		)
-		(stroke
-			(width 0)
-			(type default)
-		)
-	)
-	(wire
-		(pts
 			(xy 135.89 88.9) (xy 135.89 91.44)
 		)
@@
 	(wire
 		(pts
-			(xy 81.28 71.12) (xy 81.28 85.09)
-		)
-		(stroke
-			(width 0)
-			(type default)
-		)
-	)
-	(wire
-		(pts
 			(xy 193.04 64.77) (xy 198.12 64.77)
 		)
@@
 	(wire
 		(pts
-			(xy 90.17 66.04) (xy 74.93 66.04)
-		)
-		(stroke
-			(width 0)
-			(type default)
-		)
-	)
-	(wire
-		(pts
-			(xy 81.28 71.12) (xy 90.17 71.12)
-		)
-		(stroke
-			(width 0)
-			(type default)
-		)
-	)
-	(wire
-		(pts
 			(xy 243.84 72.39) (xy 255.27 72.39)
 		)
@@
 	(wire
 		(pts
+			(xy 68.58 66.04) (xy 81.28 66.04)
+		)
+		(stroke
+			(width 0)
+			(type default)
+		)
+	)
+	(wire
+		(pts
+			(xy 74.93 63.5) (xy 90.17 63.5)
+		)
+		(stroke
+			(width 0)
+			(type default)
+		)
+	)
+	(wire
+		(pts
 			(xy 30.48 46.99) (xy 30.48 49.53)
 		)
@@
 	(wire
 		(pts
+			(xy 74.93 63.5) (xy 74.93 80.01)
+		)
+		(stroke
+			(width 0)
+			(type default)
+		)
+	)
+	(wire
+		(pts
 			(xy 81.28 36.83) (xy 81.28 43.18)
 		)
@@
 	(wire
 		(pts
-			(xy 68.58 71.12) (xy 81.28 71.12)
+			(xy 68.58 71.12) (xy 78.74 71.12)
 		)
 		(stroke
@@
 	(wire
 		(pts
+			(xy 33.02 85.09) (xy 33.02 92.71)
+		)
+		(stroke
+			(width 0)
+			(type default)
+		)
+	)
+	(wire
+		(pts
 			(xy 205.74 69.85) (xy 204.47 69.85)
 		)
@@
 	(wire
 		(pts
-			(xy 33.02 63.5) (xy 33.02 85.09)
-		)
-		(stroke
-			(width 0)
-			(type default)
-		)
-	)
-	(wire
-		(pts
 			(xy 205.74 74.93) (xy 193.04 74.93)
 		)
 		(stroke
+			(width 0)
+			(type default)
+		)
+	)
+	(wire
+		(pts
+			(xy 81.28 66.04) (xy 81.28 85.09)
+		)
+		(stroke
+			(width 0)
+			(type default)
+		)
+	)
+	(wire
+		(pts
+			(xy 33.02 92.71) (xy 78.74 92.71)
+		)
+		(stroke
