File: STMRocket - EDA/STMRocket - KiCad Project/STMRocket.kicad_pcb (KiCad board)
At the start: 4 copper layers, 50 x 80 mm, 70 parts, among them J1 BATT XT30, J2 USB_B_Micro, J3 PYRO, J4 PYRO ARM, J5 SWD, J6 Micro_SD_Card, Q1 GSFC02A05, Q2 FDMC7692, U1 STM32F103C8T6, U2 ICM-42670-P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

Commit message: pcb update and bom
Parts:
- added H1: MountingHole, MountingHole:MountingHole_2.2mm_M2, F.Cu at (2.48, 2.48)
- added H2: MountingHole, MountingHole:MountingHole_2.2mm_M2, F.Cu at (2.48, 8.43)
- added H3: MountingHole, MountingHole:MountingHole_2.2mm_M2, F.Cu at (2.48, 14.4)
- added H4: MountingHole, MountingHole:MountingHole_2.2mm_M2, F.Cu at (2.48, 20.3)
- added H5: MountingHole, MountingHole:MountingHole_2.2mm_M2, F.Cu at (2.48, 26.3)
- moved D6 203.9 mm to (248.0, 70.1), turned to 90 degrees
- moved U4 203.9 mm to (237.0, 107.8), turned to 90 degrees
- moved C3 198.5 mm to (247.8, 62.8), turned to -90 degrees
- moved C2 198.5 mm to (247.8, 59.0), turned to 90 degrees
- moved D7 191.9 mm to (248.0, 75.9), turned to -90 degrees
- moved C5 189.3 mm to (244.4, 55.8), turned to 180 degrees
- moved C12 186.6 mm to (233.2, 103.5), turned to 90 degrees
- moved C22 186.1 mm to (233.2, 105.8), turned to -90 degrees
- moved U6 184.3 mm to (244.1, 59.0), turned to 180 degrees
- moved J5 184.2 mm to (244.8, 68.7)
- moved C26 182.4 mm to (235.4, 68.1), turned to 90 degrees
- moved C25 182.2 mm to (235.4, 70.2), turned to 90 degrees
- moved C21 181.1 mm to (226.2, 116.5), turned to -90 degrees
- moved L1 180.2 mm to (244.1, 62.8)
- moved Q1 179.6 mm to (244.2, 52.5), turned to 90 degrees
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Connections:
- C13 pad 1: GND -> Net-(U1-BOOT0)
- U1 pad 39: IMU_FSYNC -> IMU_INT2
- U1 pad 40: IMU_INT1 -> IMU_FSYNC
- U1 pad 41: IMU_INT2 -> IMU_INT1
- U5 pad 3: +3.3V -> STM_MISO
- U5 pad 4: STM_MISO -> STM_SCK
- U5 pad 5: STM_SCK -> +3.3V
Routing:
- net +3.3V: track 18.2 -> 94.3 mm, vias 2 -> 15
- net GND: track 29.9 -> 72.9 mm, vias 16 -> 65
- net STM_SWDIO: track 0.00 -> 33.3 mm
- net Net-(J6-SHIELD): track 0.00 -> 32.6 mm
- net STM_SWCLK: track 0.00 -> 31.0 mm
- net IMU_INT2: track 0.00 -> 24.3 mm
- net STM_SCL: track 0.00 -> 23.9 mm, vias 0 -> 3
- net STM_SDA: track 0.00 -> 23.3 mm
- net ~{CS}_SD: track 0.00 -> 18.6 mm, vias 0 -> 1
- net STM_MISO: track 0.00 -> 17.9 mm, vias 0 -> 1
- net PYRO_GATE: track 0.00 -> 17.2 mm
- net Net-(D4-K): track 0.00 -> 15.1 mm
- net IMU_FSYNC: track 0.00 -> 14.6 mm
- net Net-(D3-K): track 0.00 -> 13.6 mm
- net STM_SCK: track 0.00 -> 11.8 mm
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Other:
- board text added: "3V3"
- board text added: "CLK"
- board text added: "GND"
- board text added: "IO"

Commit message: PCB finished
Parts:
- removed the H1 at (2.48, 2.48)
- removed the H2 at (2.48, 8.43)
- removed the H3 at (2.48, 14.4)
- removed the H4 at (2.48, 20.3)
- removed H5: MountingHole, MountingHole:MountingHole_2.2mm_M2
- moved C7 166.0 mm to (57.0, 92.5), turned to -90 degrees
- moved C20 165.8 mm to (57.0, 89.5), turned to 90 degrees
- moved U5 162.7 mm to (55.5, 81.0), turned to 0 degrees
- moved C21 151.4 mm to (76.2, 96.2)
- moved J6 151.4 mm to (67.2, 91.6)
- moved H3 151.3 mm to (54.0, 96.0)
- moved H4 151.3 mm to (96.0, 96.0)
- moved C25 150.8 mm to (84.9, 60.2)
- moved C26 150.8 mm to (84.9, 58.1)
- moved U3 150.8 mm to (82.4, 59.2)
- moved C13 150.8 mm to (69.7, 59.9)
- moved R2 150.8 mm to (68.5, 61.2)
- moved C1 150.7 mm to (72.2, 41.5)
- moved C10 150.7 mm to (59.4, 73.6)
- moved C11 150.7 mm to (56.0, 72.3)
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Routing:
- net ~{WP}_FLASH: track 0.00 -> 65.1 mm, vias 0 -> 2
- net ~{CS}_FLASH: track 0.00 -> 55.3 mm, vias 0 -> 2
- net STM_SCK: track 11.8 -> 66.9 mm, vias 0 -> 4
- net STM_MOSI: track 11.8 -> 64.2 mm, vias 0 -> 4
- net STM_MISO: track 17.9 -> 68.9 mm, vias 1 -> 4
- net ~{HOLD}_FLASH: track 0.00 -> 43.6 mm, vias 0 -> 2
- net ~{CS}_SD: track 18.6 -> 50.2 mm, vias 1 -> 0
- net IMU_INT1: track 11.1 -> 38.3 mm
- net IMU_FSYNC: track 14.6 -> 34.7 mm
- net STM_SCL: track 23.9 -> 39.9 mm, vias 3 -> 2
- net IMU_INT2: track 24.3 -> 40.0 mm
- net PYRO_GATE: track 17.2 -> 2.55 mm
- net STM_SDA: track 23.3 -> 35.1 mm, vias 0 -> 2
- net +3.3V: track 94.3 -> 99.8 mm, vias 15 -> 22
- net Net-(D5-A): track 3.13 -> 5.43 mm
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Other:
- board size 50 x 80 mm -> 50 x 75 mm

Commit message: Final PCB revision
Parts:
- moved C1 79.1 mm to (147.2, 66.5)
- moved C11 79.1 mm to (131.1, 97.3)
- moved C17 79.1 mm to (146.2, 101.6)
- moved C25 79.1 mm to (159.9, 85.2)
- moved C27 79.1 mm to (139.2, 100.5)
- moved C4 79.1 mm to (158.3, 99.8)
- moved C5 79.1 mm to (169.4, 65.8)
- moved C6 79.1 mm to (166.2, 99.5)
- moved D6 79.1 mm to (173.0, 80.1)
- moved J2 79.1 mm to (172.1, 94.0)
- moved J3 79.1 mm to (141.8, 54.6)
- moved R8 79.1 mm to (147.7, 85.5)
- moved U3 79.1 mm to (157.4, 84.2)
- moved C12 79.1 mm to (158.5, 118.9)
- moved C14 79.1 mm to (141.3, 89.1)
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Other:
- outline, holes or cut-outs redrawn
- board text added: "Edward Sicoe 2025"
- board text added: "STMRocket"
- board text added: "https://github.com/esicoe/STMRocket"

Commit message: Final - PCB, Man. Files & BOM
Routing:
- net GND: track 72.3 -> 73.6 mm, vias 68 -> 69
Changed lines of the file:
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@@
 			(disableapertmacros no)
 			(usegerberextensions no)
-			(usegerberattributes yes)
+			(usegerberattributes no)
 			(usegerberadvancedattributes yes)
 			(creategerberjobfile yes)
@@
 			(plotframeref no)
 			(mode 1)
-			(useauxorigin no)
+			(useauxorigin yes)
 			(hpglpennumber 1)
 			(hpglpenspeed 20)
@@
 			(drillshape 0)
 			(scaleselection 1)
-			(outputdirectory "../Manufacturing Files/")
+			(outputdirectory "C:/Users/sicoe/OneDrive/Desktop/Project - STMRocket/STMRocket - Manufacturing/")
 		)
 	)
@@
 		(tags "capacitor")
 		(property "Reference" "C8"
-			(at 0 -2 180)
+			(at 2.275 0 180)
 			(layer "F.SilkS")
 			(effects
@@
 		(tags "D_SOD-123F")
 		(property "Reference" "D2"
-			(at 3.75 0 90)
+			(at 3 0 180)
 			(layer "F.SilkS")
 			(effects
@@
 		(tags "capacitor")
 		(property "Reference" "C11"
-			(at 0 -1.16 0)
+			(at 0 -1.26 0)
 			(layer "F.SilkS")
 			(effects
@@
 		(tags "TSOT TO_SOT_SMD")
 		(property "Reference" "U6"
-			(at 2.31 2.25 0)
+			(at 3.31 2.25 0)
 			(layer "F.SilkS")
 			(effects
@@
 		(tags "SOT TO_SOT_SMD")
 		(property "Reference" "Q1"
-			(at 1.78 1.85 180)
+			(at 0.04 3 180)
 			(layer "F.SilkS")
 			(effects
@@
 		(tags "capacitor")
 		(property "Reference" "C3"
-			(at 2.5 -1.25 0)
+			(at 3 -1 0)
 			(layer "F.SilkS")
 			(effects
@@
 		(tags "capacitor")
 		(property "Reference" "C5"
-			(at -2.575 0 0)
+			(at 2.675 0.25 0)
 			(layer "F.SilkS")
 			(effects
@@
 		(tags "capacitor")
 		(property "Reference" "C2"
-			(at 2.5 1.25 180)
+			(at 3.25 0 180)
 			(layer "F.SilkS")
 			(effects
@@
 		(tags "D_SOD-123F")
 		(property "Reference" "D3"
-			(at -0.127 -1.905 90)
+			(at 0 -2.22 180)
 			(layer "F.SilkS")
 			(effects
@@
 		)
 	)
+	(dimension
+		(type orthogonal)
+		(layer "F.Cu")
+		(pts
+			(xy 125 50) (xy 175 50)
+		)
+		(height -6)
+		(orientation 0)
+		(format
+			(prefix "")
+			(suffix "")
+			(units 3)
+			(units_format 0)
+			(precision 4)
+			(suppress_zeroes yes)
+		)
+		(style
+			(thickness 0.2)
+			(arrow_length 1.27)
+			(text_position_mode 0)
+			(arrow_direction outward)
+			(extension_height 0.58642)
+			(extension_offset 0.5)
+			(keep_text_aligned yes)
+		)
+		(gr_text "50"
+			(at 150 42.2 0)
+			(layer "F.Cu")
+			(effects
+				(font
+					(size 1.5 1.5)
+					(thickness 0.3)
+				)
+			)
+		)
+	)
+	(dimension
+		(type orthogonal)
+		(layer "F.Cu")
+		(pts
+			(xy 175 50) (xy 175 125)
+		)
+		(height 5.75)
+		(orientation 1)
+		(format
+			(prefix "")
+			(suffix "")
+			(units 3)
+			(units_format 0)
+			(precision 4)
+			(suppress_zeroes yes)
+		)
+		(style
+			(thickness 0.2)
+			(arrow_length 1.27)
+			(text_position_mode 0)
+			(arrow_direction outward)
+			(extension_height 0.58642)
+			(extension_offset 0.5)
+			(keep_text_aligned yes)
+		)
+		(gr_text "75"
+			(at 178.95 87.5 90)
+			(layer "F.Cu")
+			(effects
+				(font
+					(size 1.5 1.5)
+					(thickness 0.3)
+				)
+			)
+		)
+	)
 	(segment
 		(start 165.23 119.7)
@@
 	)
 	(segment
+		(start 129.5 97.25)
+		(end 129.51 97.26)
+		(width 0.25)
+		(layer "F.Cu")
+		(net 1)
+	)
+	(segment
 		(start 146.72 101.03)
 		(end 146.5 100.81)
@@
 	)
 	(segment
-		(start 130.57 96.32)
+		(start 129.51 97.26)
 		(end 130.57 97.26)
 		(width 0.25)
@@
 	)
 	(via
-		(at 130.57 96.32)
+		(at 129.5 97.25)
 		(size 0.6)
 		(drill 0.3)
@@
 	)
 	(segment
-		(start 138.75 87.25)
-		(end 138.75 85.75)
-		(width 0.25)
+		(start 148.65 58.1)
+		(end 150.25 58.1)
+		(width 0.4)
 		(layer "F.Cu")
 		(net 10)
@@
 	)
 	(segment
+		(start 138.75 87.25)
+		(end 137.5 87.25)
+		(width 0.25)
+		(layer "F.Cu")
+		(net 10)
+	)
+	(segment
 		(start 145.21 83.04)
 		(end 145.25 83)
@@
 	)
 	(via
+		(at 148.65 58.1)
+		(size 0.6)
+		(drill 0.3)
+		(layers "F.Cu" "B.Cu")
+		(net 10)
+	)
+	(via
 		(at 154.25 69.25)
 		(size 0.6)
@@
 	)
 	(via
-		(at 138.75 85.75)
+		(at 137.5 87.25)
 		(size 0.6)
 		(drill 0.3)
